File: DRV2605.sch (EAGLE design)
At the start: 18 parts, among them U2 BNO080, Y1 32.768kHz

Commit message: complete No SPI
Parts:
- removed J5: (no value), SparkFun-Connectors:CONN_01PTH_NO_SILK_YES_STOP
- added J3: BM06B-SRSS-TB, SparkFun-Connectors:JST_6_PIN_HORIZONTAL
- added U$1, U$2: SMD_PIN_1, yhtomit-single SMD pin:SMD_PIN_1
- added U$3, U$4: PH1X1, pel_hdr:PH1X1
- JP1, JP2: value JUMPER-SMT_3_NO_SILK -> JUMPER_3PLACE_1NC_XTRA_SMALL; device SparkFun-Jumpers:JUMPER-SMT_3_NO_SILK -> yhtomit_jumpers:JUMPER_3PLACE_1NC_XTRA_SMALL
- SJ2: value SOLDERJUMPERNO -> JUMPER_2PLACE_NO_XTRA_SMALL; device SparkFun:SOLDERJUMPERNO -> yhtomit_jumpers:JUMPER_2PLACE_NO_XTRA_SMALL
Connections:
- new net MOTOR+: J3A.5, U$1.P$1, U$3.2
- new net MOTOR-: J3A.4, U$2.P$1, U$4.2
- net !BOOT: no longer J5.1
- net 3.3V: now also J3A.1, JP2.1; no longer JP2.3
- net GND: now also J3A.6, JP2.3; no longer JP2.1
- net SCL/SCK/RX: now also J3A.2
- net SDA/MISO/TX: now also J3A.3
Other:
- note added: "Default, nothing is set. Solder both to GND to use i2C"
- note removed: "The default is I2C"

Commit message: SPI connector done
Parts:
- removed J3: BM06B-SRSS-TB, SparkFun-Connectors:JST_6_PIN_HORIZONTAL
- added U$6: 10&6_JSTCONNECTOR_FINGERS, yhtomit_connectors:10&6_JSTCONNECTOR_FINGERS
Connections:
- net !CS: now also U$6.1
- net !INT: now also U$6.3
- net !RST: now also U$6.4
- net 3.3V: now also U$6.5; no longer J3A.1
- net ADDR/MOSI: now also U$6.2
- net GND: now also U$6.P$4; no longer J3A.6
- net MOTOR+: now also U$6.P$3; no longer J3A.5
- net MOTOR-: now also U$6.P$2; no longer J3A.4
- net SCL/SCK/RX: now also U$6.6; no longer J3A.2
- net SDA/MISO/TX: now also U$6.P$1; no longer J3A.3
Changed lines of the file:
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@@
 <part name="JP1" library="yhtomit_jumpers" deviceset="JUMPER_3PLACE_1NC_XTRA_SMALL" device=""/>
 <part name="JP2" library="yhtomit_jumpers" deviceset="JUMPER_3PLACE_1NC_XTRA_SMALL" device=""/>
-<part name="J3" library="SparkFun-Connectors" deviceset="JST_6_PIN_HORIZONTAL" device="" value="BM06B-SRSS-TB"/>
 <part name="U$1" library="yhtomit-single SMD pin" deviceset="SMD_PIN_1" device=""/>
 <part name="U$2" library="yhtomit-single SMD pin" deviceset="SMD_PIN_1" device=""/>
 <part name="U$3" library="pel_hdr" deviceset="PH1X1" device=""/>
 <part name="U$4" library="pel_hdr" deviceset="PH1X1" device=""/>
+<part name="U$6" library="yhtomit_connectors" deviceset="10&amp;6_JSTCONNECTOR_FINGERS" device=""/>
 </parts>
 <sheets>
@@
 <instance part="JP1" gate="G$1" x="250.19" y="229.87"/>
 <instance part="JP2" gate="G$1" x="265.43" y="229.87" rot="R180"/>
-<instance part="J3" gate="A" x="190.5" y="153.67"/>
 <instance part="U$1" gate="G$1" x="148.59" y="160.02"/>
 <instance part="U$2" gate="G$1" x="148.59" y="148.59"/>
 <instance part="U$3" gate="G$1" x="116.84" y="158.75"/>
 <instance part="U$4" gate="G$1" x="116.84" y="149.86"/>
+<instance part="U$6" gate="G$1" x="190.5" y="153.67"/>
 </instances>
 <busses>
@@
 </segment>
 <segment>
-<pinref part="J3" gate="A" pin="1"/>
 <wire x1="195.58" y1="148.59" x2="201.93" y2="148.59" width="0.1524" layer="91"/>
 <label x="200.66" y="148.59" size="1.778" layer="95"/>
+<pinref part="U$6" gate="G$1" pin="5"/>
 </segment>
 <segment>
@@
 </segment>
 <segment>
-<pinref part="J3" gate="A" pin="6"/>
 <wire x1="195.58" y1="161.29" x2="201.93" y2="161.29" width="0.1524" layer="91"/>
 <label x="200.66" y="161.29" size="1.778" layer="95"/>
+<pinref part="U$6" gate="G$1" pin="P$4"/>
 </segment>
 <segment>
@@
 <junction x="95.25" y="214.63"/>
 </segment>
+<segment>
+<pinref part="U$6" gate="G$1" pin="2"/>
+<wire x1="195.58" y1="140.97" x2="200.66" y2="140.97" width="0.1524" layer="91"/>
+<label x="200.66" y="140.97" size="1.778" layer="95"/>
+</segment>
 </net>
 <net name="!BOOT" class="0">
@@
 <label x="143.51" y="204.47" size="1.27" layer="95" rot="R180" xref="yes"/>
 </segment>
+<segment>
+<pinref part="U$6" gate="G$1" pin="1"/>
+<wire x1="195.58" y1="138.43" x2="200.66" y2="138.43" width="0.1524" layer="91"/>
+<label x="200.66" y="138.43" size="1.778" layer="95"/>
+</segment>
 </net>
 <net name="!INT" class="0">
@@
 <wire x1="148.59" y1="207.01" x2="143.51" y2="207.01" width="0.1524" layer="91"/>
 <label x="143.51" y="207.01" size="1.27" layer="95" rot="R180" xref="yes"/>
+</segment>
+<segment>
+<pinref part="U$6" gate="G$1" pin="3"/>
+<wire x1="195.58" y1="143.51" x2="201.93" y2="143.51" width="0.1524" layer="91"/>
+<label x="200.66" y="143.51" size="1.778" layer="95"/>
 </segment>
 </net>
@@
 </segment>
 <segment>
-<pinref part="J3" gate="A" pin="2"/>
 <wire x1="195.58" y1="151.13" x2="201.93" y2="151.13" width="0.1524" layer="91"/>
 <label x="200.66" y="151.13" size="1.778" layer="95"/>
+<pinref part="U$6" gate="G$1" pin="6"/>
 </segment>
 </net>
@@
 </segment>
 <segment>
-<pinref part="J3" gate="A" pin="3"/>
 <wire x1="195.58" y1="153.67" x2="201.93" y2="153.67" width="0.1524" layer="91"/>
 <label x="200.66" y="153.67" size="1.778" layer="95"/>
+<pinref part="U$6" gate="G$1" pin="P$1"/>
 </segment>
 </net>
@@
 <junction x="189.23" y="222.25"/>
 <label x="191.77" y="222.25" size="1.27" layer="95" xref="yes"/>
+</segment>
+<segment>
+<pinref part="U$6" gate="G$1" pin="4"/>
+<wire x1="195.58" y1="146.05" x2="201.93" y2="146.05" width="0.1524" layer="91"/>
+<label x="200.66" y="146.05" size="1.778" layer="95"/>
 </segment>
 </net>
@@
 </segment>
 <segment>
-<pinref part="J3" gate="A" pin="5"/>
 <wire x1="195.58" y1="158.75" x2="201.93" y2="158.75" width="0.1524" layer="91"/>
 <label x="200.66" y="158.75" size="1.778" layer="95"/>
+<pinref part="U$6" gate="G$1" pin="P$3"/>
 </segment>
 </net>
@@
 </segment>
 <segment>
-<pinref part="J3" gate="A" pin="4"/>
 <wire x1="195.58" y1="156.21" x2="201.93" y2="156.21" width="0.1524" layer="91"/>
 <label x="200.66" y="156.21" size="1.778" layer="95"/>
-</segment>
-</net>
+<pinref part="U$6" gate="G$1" pin="P$2"/>
+</segment>
+</net>

Commit message: Complete
Other:
- moved on the sheet: C1, C2, C3, C4, C5, JP1, JP2, R1, R10, R12, R13, R3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
