File: DRV2605.brd (EAGLE design)
At the start: 11 x 19.8 mm, 18 parts, among them U2 BNO080, Y1 32.768kHz

Commit message: complete No SPI
Parts:
- removed J5: (no value), SparkFun-Connectors:1X01_NO_SILK
- added J3: BM06B-SRSS-TB, SparkFun-Connectors:JST-6-SMD-HORI-1.0MM
- added U$1, U$2: SMD_PIN_1, yhtomit-single SMD pin:SMD_PIN
- added U$3, U$4: PH1X1, pel_hdr:PH005-1-1
- JP1, JP2: value JUMPER-SMT_3_NO_SILK -> JUMPER_3PLACE_1NC_XTRA_SMALL; device SparkFun-Jumpers:SMT-JUMPER_3_NO_SILK -> yhtomit_jumpers:XTRA_SMAL_JUMPER_3_1_NC
- SJ2: value (none) -> JUMPER_2PLACE_NO_XTRA_SMALL; device SparkFun:SJ_2S-NO -> yhtomit_jumpers:XTRA_SMALLJUMPER_NO
- moved JP2 45.9 mm to (2.47, 4.81), flipped to the bottom, turned to 90 degrees
- moved JP1 40.4 mm to (4.02, 4.83), flipped to the bottom, turned to 90 degrees
- moved SJ2 5.41 mm to (10.5, 8.89), flipped to the bottom, turned to 0 degrees
- moved R3 5.14 mm to (10.2, 7.28), flipped to the bottom
- moved R1 5.06 mm to (7.55, 5.18), flipped to the bottom
- moved C1 4.81 mm to (5.92, 4.87), flipped to the bottom
- moved R9 4.76 mm to (9.73, 5.18), flipped to the bottom
- moved R10 4.67 mm to (8.61, 5.18), flipped to the bottom
- moved C4 4.37 mm to (3.24, 9.19), flipped to the bottom, turned to 270 degrees
- moved R12 2.75 mm to (7.23, 11.5), flipped to the bottom, turned to 0 degrees
- moved R13 2.21 mm to (7.21, 10.5), flipped to the bottom, turned to 0 degrees
- moved U2 2.07 mm to (5.85, 9.98)
- moved R6 2.05 mm to (1.76, 8.80)
- moved Y1 1.65 mm to (5.36, 13.6)
- moved C2 1.51 mm to (2.14, 9.20), flipped to the bottom
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Connections:
- new net MOTOR+: J3.5, U$1.P$2, U$3.1
- new net MOTOR-: J3.4, U$2.P$2, U$4.1
- net !BOOT: no longer J5.1
- net 3.3V: now also J3.1, JP2.1; no longer JP2.3
- net GND: now also J3.6, JP2.3; no longer JP2.1
- net SCL/SCK/RX: now also J3.2
- net SDA/MISO/TX: now also J3.3
Routing:
- net 3.3V: track 0.00 -> 36.4 mm, vias 0 -> 2
- net MOTOR+: track 0.00 -> 27.3 mm, vias 0 -> 1
- net MOTOR-: track 0.00 -> 24.2 mm, vias 0 -> 1
- net SDA/MISO/TX: track 0.00 -> 21.5 mm, vias 0 -> 2
- net SCL/SCK/RX: track 0.00 -> 20.3 mm, vias 0 -> 2
- net PS1: track 0.00 -> 5.58 mm, vias 0 -> 1
- net N$2: track 0.00 -> 4.87 mm
- net S_SDA: track 0.00 -> 4.16 mm, vias 0 -> 1
- net PS0/WAKE: track 0.00 -> 3.87 mm, vias 0 -> 1
- net N$1: track 0.00 -> 3.79 mm
- net ADDR/MOSI: track 0.00 -> 3.62 mm, vias 0 -> 1
- net S_SCL: track 0.00 -> 3.42 mm, vias 0 -> 1
- net CAP: track 0.00 -> 3.41 mm, vias 0 -> 1
- net !RST: track 0.00 -> 3.24 mm, vias 0 -> 1
- net !BOOT: track 0.00 -> 3.18 mm
- added copper zone on layer 16, net GND
Other:
- board size 11 x 19.8 mm -> 12 x 15 mm

Commit message: SPI connector done
Parts:
- removed J3: BM06B-SRSS-TB, SparkFun-Connectors:JST-6-SMD-HORI-1.0MM
- added U$6: 10&6_JSTCONNECTOR_FINGERS, yhtomit_connectors:10&4_HORIZONTAL_JST_CONN
Connections:
- net !CS: now also U$6.1
- net !INT: now also U$6.3
- net !RST: now also U$6.4
- net 3.3V: now also U$6.5; no longer J3.1
- net ADDR/MOSI: now also U$6.2
- net GND: now also U$6.10; no longer J3.6
- net MOTOR+: now also U$6.9; no longer J3.5
- net MOTOR-: now also U$6.8; no longer J3.4
- net SCL/SCK/RX: now also U$6.6; no longer J3.2
- net SDA/MISO/TX: now also U$6.7; no longer J3.3
Routing:
- net MOTOR+: track 27.3 -> 24.1 mm
- net SCL/SCK/RX: track 20.3 -> 22.8 mm
- net SDA/MISO/TX: track 21.5 -> 23.9 mm
- net MOTOR-: track 24.2 -> 22.5 mm
- net 3.3V: track 36.4 -> 35.9 mm

Commit message: Complete awaiting DRC
Parts:
- moved Y1 0.20 mm to (5.36, 13.8)
Routing:
- net !CS: track 0.00 -> 6.80 mm
- net ADDR/MOSI: track 3.62 -> 7.90 mm
- net !INT: track 0.00 -> 3.59 mm
- net !RST: track 3.24 -> 5.27 mm
- net S_SCL: track 3.42 -> 2.81 mm

Commit message: Complete
Parts:
- moved R10 0.52 mm to (9.13, 5.18)
- moved C1 0.52 mm to (6.44, 4.87)
- moved JP1 0.52 mm to (4.54, 4.83)
- moved R1 0.52 mm to (8.07, 5.18)
- moved R13 0.52 mm to (7.73, 10.5)
- moved U$1 0.52 mm to (7.65, 13.5)
- moved U2 0.52 mm to (6.37, 9.98)
- moved C2 0.52 mm to (2.66, 9.20)
- moved C5 0.52 mm to (3.32, 13.5)
- moved JP2 0.52 mm to (2.99, 4.81)
- moved U$4 0.52 mm to (1.52, 13.9)
- moved R6 0.52 mm to (2.28, 8.80)
- moved C3 0.52 mm to (8.36, 13.5)
- moved C4 0.52 mm to (3.76, 9.19)
- moved R12 0.52 mm to (7.75, 11.5)
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Other:
- board text added: "+"
- board text added: "_"

Commit message: Complete
Parts:
- moved R10 0.52 mm to (8.61, 5.18)
- moved C1 0.52 mm to (5.92, 4.87)
- moved JP1 0.52 mm to (4.02, 4.83)
- moved R1 0.52 mm to (7.55, 5.18)
- moved R13 0.52 mm to (7.21, 10.5)
- moved U$1 0.52 mm to (7.13, 13.5)
- moved U2 0.52 mm to (5.85, 9.98)
- moved C2 0.52 mm to (2.14, 9.20)
- moved C5 0.52 mm to (2.80, 13.5)
- moved JP2 0.52 mm to (2.47, 4.81)
- moved U$4 0.52 mm to (1.00, 13.9)
- moved R6 0.52 mm to (1.76, 8.80)
- moved C3 0.52 mm to (7.84, 13.5)
- moved C4 0.52 mm to (3.24, 9.19)
- moved R12 0.52 mm to (7.23, 11.5)
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