File: DRV2605_USB.sch (EAGLE design)
At the start: 23 parts, among them U2 BNO080, Y1 32.768kHz

Commit message: USB port added; motor connectors removed
Parts:
- removed J1: (no value), SparkFun-Connectors:USB_MICRO-BREDUCED_PASTE
Changed lines of the file:
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@@
 <part name="U$4" library="pel_hdr" deviceset="PH1X1" device=""/>
 <part name="U$6" library="yhtomit_connectors" deviceset="10&amp;6_JSTCONNECTOR_FINGERS" device=""/>
-<part name="J1" library="SparkFun-Connectors" library_urn="urn:adsk.eagle:library:513" deviceset="USB_MICRO-B" device="REDUCED_PASTE" package3d_urn="urn:adsk.eagle:package:38239/1"/>
 </parts>
 <sheets>
@@
 <instance part="U$4" gate="G$1" x="132.08" y="35.56"/>
 <instance part="U$6" gate="G$1" x="205.74" y="39.37"/>
-<instance part="J1" gate="G$1" x="299.72" y="88.9"/>
 </instances>
 <busses>
